File: finalproj/schematic/schematic.kicad_sch (KiCad schematic)
At the start: 55 parts, among them U1 74HC165, U2 74HC165, U3 74HC165, U4 74HC165

Commit message: edited schematic for rotary switches
Parts:
- added U5, U6: ~, symbol ky_040:KY_040
Connections:
- net GND: now also U5.5 (GND), U6.5 (GND)
- net at A1.5 (+5V), R1.2, R10.2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: now also U5.4 (Vcc), U6.4 (Vcc)
- net at A1.20 (D5): now also U5.1 (CLK)
- net at A1.21 (D6): now also U5.2 (DT)
- net at A1.22 (D7): now also U6.1 (CLK)
- net at A1.23 (D8): now also U6.2 (DT)
- no-connect marks 63 -> 61
